Commit message: urdf damping update for GAZEBO jerk -- 여전히 떨림.

File: dsr_description/config/macro.gazebo.xacro (robot description, xacro)
@@ -76,4 +76,47 @@
 			<minDepth>0.001</minDepth>
 		</gazebo>
+		<!-- Joint-specific Gazebo dynamics -->
+		<gazebo reference="joint1">
+			<implicitSpringDamper>true</implicitSpringDamper>
+			<springStiffness>0</springStiffness>
+			<springReference>0</springReference>
+			<damping>10.0</damping>
+			<friction>1.0</friction>
+		</gazebo>
+		<gazebo reference="joint2">
+			<implicitSpringDamper>true</implicitSpringDamper>
+			<springStiffness>0</springStiffness>
+			<springReference>0</springReference>
+			<damping>10.0</damping>
+			<friction>1.0</friction>
+		</gazebo>
+		<gazebo reference="joint3">
+			<implicitSpringDamper>true</implicitSpringDamper>
+			<springStiffness>0</springStiffness>
+			<springReference>0</springReference>
+			<damping>5.0</damping>
+			<friction>0.8</friction>
+		</gazebo>
+		<gazebo reference="joint4">
+			<implicitSpringDamper>true</implicitSpringDamper>
+			<springStiffness>0</springStiffness>
+			<springReference>0</springReference>
+			<damping>3.0</damping>
+			<friction>0.5</friction>
+		</gazebo>
+		<gazebo reference="joint5">
+			<implicitSpringDamper>true</implicitSpringDamper>
+			<springStiffness>0</springStiffness>
+			<springReference>0</springReference>
+			<damping>3.0</damping>
+			<friction>0.5</friction>
+		</gazebo>
+		<gazebo reference="joint6">
+			<implicitSpringDamper>true</implicitSpringDamper>
+			<springStiffness>0</springStiffness>
+			<springReference>0</springReference>
+			<damping>2.0</damping>
+			<friction>0.3</friction>
+		</gazebo>
 		<!-- ros_control plugin -->
 		<gazebo>

File: dsr_description/xacro/macro.m1509.white.xacro (robot description, xacro)
@@ -34,5 +34,5 @@
 			<axis xyz="0 0 1" />
 			<limit effort="346" lower="-6.2832" upper="6.2832" velocity="2.618"/>
-			<dynamics friction="0" />
+			<dynamics damping="10.0" friction="1.0" />
 		</joint>
 		<link name="link1">
@@ -64,5 +64,5 @@
 			<axis xyz="0 0 1" />
 			<limit effort="346" lower="-6.2832" upper="6.2832" velocity="2.618"/>
-			<dynamics friction="0" />
+			<dynamics damping="10.0" friction="1.0" />
 		</joint>
 		<link name="link2">
@@ -117,5 +117,5 @@
 			<axis xyz="0 0 1" />
 			<limit effort="163" lower="-2.618" upper="2.618" velocity="3.1416"/>
-			<dynamics friction="0" />
+			<dynamics damping="5.0" friction="0.8" />
 		</joint>
 		<link name="link3">
@@ -147,5 +147,5 @@
 			<axis xyz="0 0 1" />
 			<limit effort="50" lower="-6.2832" upper="6.2832" velocity="3.927"/>
-			<dynamics friction="0" />
+			<dynamics damping="3.0" friction="0.5" />
 		</joint>
 		<link name="link4">
@@ -189,5 +189,5 @@
 			<axis xyz="0 0 1" />
 			<limit effort="50" lower="-6.2832" upper="6.2832" velocity="3.927"/>
-			<dynamics friction="0" />
+			<dynamics damping="3.0" friction="0.5" />
 		</joint>
 		<link name="link5">
@@ -219,5 +219,5 @@
 			<axis xyz="0 0 1" />
 			<limit effort="50" lower="-6.2832" upper="6.2832" velocity="3.927"/>
-			<dynamics friction="0" />
+			<dynamics damping="2.0" friction="0.3" />
 		</joint>
 		<link name="link6">
